File: Multiscope.kicad_pcb (KiCad board)
At the start: 2 copper layers, 240.7 x 139.7 mm, 72 parts, among them J2 USB_B_Micro, J3 Conn_01x01_Socket, J4 Conn_01x01_Socket, J5 Conn_01x01_Socket, J6 Conn_01x01_Socket, J7 Conn_01x01_Socket, J8 Conn_01x01_Socket, SW1 SW_Push, SW2 SW_Push, SW3 SW_Push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

Commit message: Laid out traces for display
Parts:
- added J10: Conn_01x01_Socket, Connector:Banana_Jack_1Pin, F.Cu at (80.3, 151.1)
- added J9: Conn_01x01_Socket, Connector:Banana_Jack_1Pin, F.Cu at (67.3, 151.1)
- moved D2 143.3 mm to (38.4, 99.8), turned to 90 degrees
- moved C15 119.0 mm to (31.8, 119.8), turned to 90 degrees
- moved U10 117.5 mm to (73.3, 142.5), turned to 180 degrees
- moved C14 115.3 mm to (31.5, 102.4), turned to 90 degrees
- moved J7 108.2 mm to (114.3, 151.1)
- moved J3 105.7 mm to (97.3, 151.1)
- moved J5 101.8 mm to (148.3, 151.1)
- moved C16 99.6 mm to (45.0, 97.7), turned to -90 degrees
- moved SW5 99.3 mm to (55.9, 99.3)
- moved J4 96.9 mm to (165.4, 151.1)
- moved C17 96.7 mm to (111.1, 98.0)
- moved C18 95.5 mm to (48.5, 97.6), turned to -90 degrees
- moved SW3 95.4 mm to (78.4, 136.6), turned to 180 degrees
- moved R10 95.3 mm to (34.8, 108.2), turned to 180 degrees
- moved R11 95.0 mm to (35.1, 105.2)
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Connections:
- R1 pad 1: unconnected-(R1-Pad1) -> Net-(U1-BOOT0)
- R13 pad 2: SDA -> POWER_PROBE_M
- U1 pad 59: SDA -> POWER_PROBE_M
- U10 pad 4: SDA -> POWER_PROBE_M
- U12 pad 1: ADC123_IN11 -> ADC123_IN3
- U12 pad 4: ADC123_IN11 -> ADC123_IN3
- U3 pad 1: ADC123_IN0 -> ADC123_IN11
- U4 pad 1: ADC123_IN1 -> ADC123_IN0
- U5 pad 1: ADC123_IN2 -> ADC123_IN1
- U6 pad 1: ADC123_IN3 -> ADC123_IN2
Routing:
- net LED+: track 24.9 -> 543.8 mm, vias 0 -> 8
- net POT_CS: track 0.00 -> 137.2 mm, vias 0 -> 6
- net POT_UD: track 0.00 -> 130.8 mm, vias 0 -> 8
- net ADC123_IN3: track 0.00 -> 126.0 mm
- net ADC123_IN2: track 0.00 -> 100.2 mm
- net ADC123_IN1: track 0.00 -> 82.6 mm
- net POWER_PROBE_M: track 0.00 -> 72.8 mm
- net DISPLAY_A0: track 0.00 -> 69.1 mm, vias 0 -> 3
- net DISPLAY_RST: track 0.00 -> 67.6 mm, vias 0 -> 2
- net ADC123_IN0: track 0.00 -> 63.0 mm
- net Net-(U1-NRST): track 0.00 -> 62.0 mm, vias 0 -> 2
- net DISPLAY_CS: track 0.00 -> 61.0 mm, vias 0 -> 1
- net ADC123_IN11: track 0.00 -> 46.9 mm
- net DISPLAY_SCL: track 0.00 -> 45.9 mm, vias 0 -> 2
- net POWER_PROBE_P: track 0.00 -> 45.3 mm
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Other:
- board size 240.7 x 139.7 mm -> 165.2 x 77.7 mm
- board text added: "${REFERENCE}"
